File: hardware/power-management-unit/rev-a2-layout-280x260/kicad/HomeMy_PMU_RevA.kicad_pcb (KiCad board)
At the start: 4 copper layers, 280 x 260 mm, 425 parts, among them J1 Battery M5 160A class, J10 5V logic-buck INPUT, J11 5V converter OUTPUT return, J12 External resistor bank, J13 24V lift clamp DNP, J14 Analog bank NTC, J15 Telemetry bank NTC, J16 CAN backbone IN, J17 CAN backbone OUT, J18 5V LED strip 5A, J2 Battery M5 160A class, J20 TSW-102-07-G-S, J21 TSW-105-07-G-S, J22 TSW-103-07-G-S, J23 TSW-103-07-G-S, J3 Left arm + M5 160A class, J4 Left arm return M5 160A class, J5 Right arm + M5 160A class, J6 Right arm return M5 160A class, J7 Drive 8A peak, J8 24V lift-buck INPUT, J9 12V PC-buck INPUT, Q1 100V N-MOS .99mR@25C/2.3mR@17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, Q10 100V N-MOS .99mR@25C/2.3mR@17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, Q11 Remote temperature diode, Q2 100V N-MOS .99mR@25C/2.3mR@17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, Q20 BSS138BK,215, Q21 BSS138BK,215, Q3 100V N-MOS .99mR@25C/2.3mR@17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, Q4 100V N-MOS .99mR@25C/2.3mR@17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, Q40 100V chopper NMOS, Q41 NTC healthy enables driver, Q42 Chopper gate status isolation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, Q43 Qualified fault LED power, Q44 Qualified local enable, Q5 100V N-MOS .99mR@25C/2.3mR@17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, Q6 100V N-MOS .99mR@25C/2.3mR@17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, Q7 100V N-MOS .99mR@25C/2.3mR@17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, Q8 100V N-MOS .99mR@25C/2.3mR@17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, Q9 100V N-MOS .99mR@25C/2.3mR@17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, U1 LM74930-Q1, U10 ESP32-S3-WROOM-1-N8, U11 INA228AIDGSR, U12 TLV1117LV33DCYR, U13 TCAN1042HGVDRQ1, U14 SN74AHCT1G125DBVR, U15 LT3014BIS5#TRPBF, U16 LTC2954ITS8-1#TRPBF, U17 TPS3839G33DBZR, U18 SN74LVC1G74DCUR, U19 SN74LVC2G00DCUR, U2 TPS48110-Q1, U20 SN74LVC1G14DBVR, U21 LTC6993IS6-1#TRPBF, U22 SN74LVC1G32DBVR, U23 SN74LVC1G74DCUR, U24 SN74LVC2G00DCUR, U25 SN74LVC1G11DBVR, U26 TPS3839G33DBZR, U27 SN74LVC1G74DCUR, U28 SN74LVC1G11DBVR, U29 SN74LVC1G11DBVR, U3 TPS26631 eFuse latch-off, U30 100V LDO, nominal 10V, U31 2.5V high-grade reference, U32 Independent analog chopper/OV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, U33 4A source/8A sink driver, U34 Isolated analog fault, U35 Isolated chopper active, U36 Reference qualification 12..2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, U4 TPS26631 eFuse latch-off, U5 Latched motion SYS undervolta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, U50 SN74LVC1G11DBVR, U51 TPS3431SDRBR, U53 SN74LVC1G14DBVR, U54 SN74LVC1G11DBVR, U55 SN74LVC1G74DCUR, U56 SN74LVC1G14DBVR, U57 SN74LVC1G11DBVR, U58 SN74LVC1G32DBVR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

Commit message: hardware: advance PMU A2 routing and verify remaining WIP
Routing:
- net I2C_SCL: track 60.1 -> 487.7 mm, vias 2 -> 12
- net TEMP_MAIN_ADC: track 57.4 -> 375.7 mm, vias 2 -> 14
- net SW_RESET_N: track 181.1 -> 334.9 mm, vias 6 -> 10
- net LED_DATA_3V3: track 64.7 -> 203.0 mm, vias 2 -> 11
- net BUTTON_INT_N: track 86.4 -> 215.5 mm, vias 2 -> 12
- net ESP_MOTION_RESET: track 92.8 -> 66.3 mm
- net MOTION_BUS_P: track 144.6 -> 122.9 mm, vias 227 -> 226
- net MOTION_TEMP_FLT_N: track 290.4 -> 272.8 mm
- net MOTION_FAULTS_OK: track 39.0 -> 26.0 mm
- net SYS_BUS_P: track 285.1 -> 275.4 mm
- net ESP_CHIP_EN: track 293.1 -> 284.7 mm
- net MAIN_FAULT_N: track 205.6 -> 197.9 mm
- net BATT_N: track 466.6 -> 463.3 mm
- net MOTION_FLT_N: track 290.1 -> 288.4 mm
- net CHOP_10V: track 218.0 -> 216.4 mm, vias 6 -> 5
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