File: hardware/power-management-unit/rev-a2-layout-280x260/kicad/HomeMy_PMU_RevA.kicad_pcb (KiCad board)
At the start: 4 copper layers, 280 x 260 mm, 425 parts, among them J1 Battery M5 160A class, J10 5V logic-buck INPUT, J11 5V converter OUTPUT return, J12 External resistor bank, J13 24V lift clamp DNP, J14 Analog bank NTC, J15 Telemetry bank NTC, J16 CAN backbone IN, J17 CAN backbone OUT, J18 5V LED strip 5A, J2 Battery M5 160A class, J20 TSW-102-07-G-S, J21 TSW-105-07-G-S, J22 TSW-103-07-G-S, J23 TSW-103-07-G-S, J3 Left arm + M5 160A class, J4 Left arm return M5 160A class, J5 Right arm + M5 160A class, J6 Right arm return M5 160A class, J7 Drive 8A peak, J8 24V lift-buck INPUT, J9 12V PC-buck INPUT, Q1 100V N-MOS .99mR@25C/2.3mR@17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, Q10 100V N-MOS .99mR@25C/2.3mR@17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, Q11 Remote temperature diode, Q2 100V N-MOS .99mR@25C/2.3mR@17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, Q20 BSS138BK,215, Q21 BSS138BK,215, Q3 100V N-MOS .99mR@25C/2.3mR@17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, Q4 100V N-MOS .99mR@25C/2.3mR@17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, Q40 100V chopper NMOS, Q41 NTC healthy enables driver, Q42 Chopper gate status isolation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, Q43 Qualified fault LED power, Q44 Qualified local enable, Q5 100V N-MOS .99mR@25C/2.3mR@17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, Q6 100V N-MOS .99mR@25C/2.3mR@17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, Q7 100V N-MOS .99mR@25C/2.3mR@17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, Q8 100V N-MOS .99mR@25C/2.3mR@17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, Q9 100V N-MOS .99mR@25C/2.3mR@17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, U1 LM74930-Q1, U10 ESP32-S3-WROOM-1-N8, U11 INA228AIDGSR, U12 TLV1117LV33DCYR, U13 TCAN1042HGVDRQ1, U14 SN74AHCT1G125DBVR, U15 LT3014BIS5#TRPBF, U16 LTC2954ITS8-1#TRPBF, U17 TPS3839G33DBZR, U18 SN74LVC1G74DCUR, U19 SN74LVC2G00DCUR, U2 TPS48110-Q1, U20 SN74LVC1G14DBVR, U21 LTC6993IS6-1#TRPBF, U22 SN74LVC1G32DBVR, U23 SN74LVC1G74DCUR, U24 SN74LVC2G00DCUR, U25 SN74LVC1G11DBVR, U26 TPS3839G33DBZR, U27 SN74LVC1G74DCUR, U28 SN74LVC1G11DBVR, U29 SN74LVC1G11DBVR, U3 TPS26631 eFuse latch-off, U30 100V LDO, nominal 10V, U31 2.5V high-grade reference, U32 Independent analog chopper/OV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, U33 4A source/8A sink driver, U34 Isolated analog fault, U35 Isolated chopper active, U36 Reference qualification 12..2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, U4 TPS26631 eFuse latch-off, U5 Latched motion SYS undervolta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, U50 SN74LVC1G11DBVR, U51 TPS3431SDRBR, U53 SN74LVC1G14DBVR, U54 SN74LVC1G11DBVR, U55 SN74LVC1G74DCUR, U56 SN74LVC1G14DBVR, U57 SN74LVC1G11DBVR, U58 SN74LVC1G32DBVR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

Commit message: Close remaining PMU A2 280x260 nets and pass native CAD checks
Preserve source topology, placement and rules. Record two identical clean native suites with 247 power pairs and 46 critical paths, and add a clearly unreleased manufacturing draft. Keep all release flags false: locked Mac blocks final graphical reopen verification, and physical production qualification is still open.
Routing:
- net TEMP_MOTION_ADC: track 34.4 -> 406.7 mm, vias 3 -> 14
- net CAN_STB: track 14.1 -> 231.7 mm, vias 1 -> 20
- net I2C_SDA: track 331.6 -> 493.4 mm, vias 5 -> 19
- net I2C_SCL: track 487.7 -> 482.4 mm
Other:
- board text added: "PMU A.2 280x260 DRAFT - NOT RELEASED"
- board text removed: "PMU A.2 280x260 WIP - NOT RELEASED"
